File: K410T-devboard.kicad_pcb (KiCad board)
At the start: 2 copper layers, 0 parts

Commit message: Create nano-ITX board edge, create\ FPGA quadrant-style fanout
Parts:
- added C1: C_47u_0603, antmicro-footprints:0603-cap, F.Cu at (292.4, 102.5)
- added C10: C_4u7_0402, antmicro-footprints:0402-cap, F.Cu at (299.1, 99.8)
- added C11: C_4u7_0402, antmicro-footprints:0402-cap, F.Cu at (283.7, 89.3)
- added C12: C_4u7_0402, antmicro-footprints:0402-cap, F.Cu at (295.6, 102.2)
- added C13: C_47u_0603, antmicro-footprints:0603-cap, F.Cu at (290.1, 78.7)
- added C14: C_4u7_0402, antmicro-footprints:0402-cap, F.Cu at (293.3, 78.4)
- added C15: C_47u_0603, antmicro-footprints:0603-cap, F.Cu at (295.9, 100.0)
- added C16: C_4u7_0402, antmicro-footprints:0402-cap, F.Cu at (295.8, 76.0)
- added C17: C_47u_0603, antmicro-footprints:0603-cap, F.Cu at (284.0, 87.1)
- added C18: C_47u_0603, antmicro-footprints:0603-cap, F.Cu at (286.5, 83.1)
- added C19: C_47u_0603, antmicro-footprints:0603-cap, F.Cu at (286.5, 80.7)
- added C2: C_47u_0603, antmicro-footprints:0603-cap, F.Cu at (292.6, 76.2)
- added C20: C_47u_0603, antmicro-footprints:0603-cap, F.Cu at (286.5, 78.2)
- added C21: C_47u_0603, antmicro-footprints:0603-cap, F.Cu at (290.1, 81.1)
- added C22: C_47u_0603, antmicro-footprints:0603-cap, F.Cu at (296.1, 73.7)
- added C23: C_4u7_0402, antmicro-footprints:0402-cap, F.Cu at (280.1, 93.8)
- added C24: C_47u_0603, antmicro-footprints:0603-cap, F.Cu at (280.4, 87.1)
- added C25: C_330u_KEMET_B, antmicro-footprints:KEMET_B, F.Cu at (286.1, 101.0)
- added C26: C_330u_KEMET_B, antmicro-footprints:KEMET_B, F.Cu at (280.2, 79.2)
- added C27: C_330u_KEMET_B, antmicro-footprints:KEMET_B, F.Cu at (286.2, 74.7)
- added C28: C_330u_KEMET_B, antmicro-footprints:KEMET_B, F.Cu at (280.2, 83.6)
- added C29: C_330u_KEMET_B, antmicro-footprints:KEMET_B, F.Cu at (280.2, 74.7)
- added C3: C_47u_0603, antmicro-footprints:0603-cap, F.Cu at (292.4, 100.0)
- added C4: C_47u_0603, antmicro-footprints:0603-cap, F.Cu at (292.6, 73.7)
- added C5: C_47u_0603, antmicro-footprints:0603-cap, F.Cu at (280.4, 89.5)
- added C6: C_330u_KEMET_B, antmicro-footprints:KEMET_B, F.Cu at (280.0, 101.0)
- added C7: C_4u7_0402, antmicro-footprints:0402-cap, F.Cu at (299.3, 73.5)
- added C8: C_4u7_0402, antmicro-footprints:0402-cap, F.Cu at (280.1, 91.8)
- added C9: C_4u7_0402, antmicro-footprints:0402-cap, F.Cu at (287.2, 85.3)
- added U1: XC7K410T-2FFG900I, antmicro-footprints:xc7k410t-2ffg900I, F.Cu at (210.0, 130.0)
Routing:
- net GND: track 0.00 -> 122.3 mm, vias 0 -> 173
- net VCCINT: track 0.00 -> 14.1 mm, vias 0 -> 20
- net VCCO_34: track 0.00 -> 4.95 mm, vias 0 -> 7
- net VCCO_17: track 0.00 -> 4.95 mm, vias 0 -> 7
- net VCCO_16: track 0.00 -> 4.95 mm, vias 0 -> 7
- net VCCO_33: track 0.00 -> 4.24 mm, vias 0 -> 6
- net VCCO_32: track 0.00 -> 4.24 mm, vias 0 -> 6
- net VCCO_18: track 0.00 -> 4.24 mm, vias 0 -> 6
- net VCCO_15: track 0.00 -> 4.24 mm, vias 0 -> 6
- net VCCO_14: track 0.00 -> 4.24 mm, vias 0 -> 6
- net VCCO_13: track 0.00 -> 4.24 mm, vias 0 -> 6
- net VCCO_12: track 0.00 -> 4.24 mm, vias 0 -> 6
- net VCCAUX: track 0.00 -> 3.54 mm, vias 0 -> 5
- net VCCBRAM: track 0.00 -> 2.83 mm, vias 0 -> 4
- net VCCAUX_IO_G0: track 0.00 -> 2.12 mm, vias 0 -> 3
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Other:
- board outline added: 120 x 120 mm
