File: K410T-devboard.kicad_pcb (KiCad board)
At the start: 2 copper layers, 120 x 120 mm, 241 parts, among them J1 878321412, Q1 BSS138W-7-F, Q2 BSS138W-7-F, SW1 CVS-03B, U1 XC7K410T-2FFG900I, U2 MT41K512M8DA, U3 TPD4E05U06QDQARQ1, U4 MPM54304GMN, U5 AS6C8008-55ZIN, U6 MT25QL256ABA1EW7-0SIT, U7 MPM3650GQW-Z

Commit message: Connect MGT supplies, fix FMC+ connector, export components to PCB
Parts:
- added C171: C_100n_0805_100V, antmicro-footprints:0805-cap, F.Cu at (305.5, 199.7)
- added C172: C_22u_2220_100V, antmicro-footprints:2220-cap, F.Cu at (280.4, 194.8)
- added C173: C_22u_2220_100V, antmicro-footprints:2220-cap, F.Cu at (328.8, 165.9)
- added C174: C_22u_2220_100V, antmicro-footprints:2220-cap, F.Cu at (316.3, 182.7)
- added C175: C_100n_0402_50V, antmicro-footprints:0402-cap, F.Cu at (354.2, 163.4)
- added C176: C_22u_2220_100V, antmicro-footprints:2220-cap, F.Cu at (290.0, 190.4)
- added C177: C_47u_16V_1206, antmicro-footprints:1206-cap, F.Cu at (294.9, 195.9)
- added C178: C_47u_16V_1206, antmicro-footprints:1206-cap, F.Cu at (305.4, 188.6)
- added C179: C_47u_16V_1206, antmicro-footprints:1206-cap, F.Cu at (279.4, 200.0)
- added C180: C_100n_0402, antmicro-footprints:0402-cap, F.Cu at (335.2, 181.9)
- added C181: C_100n_0402, antmicro-footprints:0402-cap, F.Cu at (320.0, 194.2)
- added C182: C_100n_0402, antmicro-footprints:0402-cap, F.Cu at (350.3, 166.3)
- added C183: C_1u_0603_25V, antmicro-footprints:0603-cap, F.Cu at (332.0, 179.8)
- added C184: C_1u_0603_25V, antmicro-footprints:0603-cap, F.Cu at (340.7, 173.7)
- added C185: C_1u_0603_25V, antmicro-footprints:0603-cap, F.Cu at (313.5, 200.9)
- added C186: C_100n_0402, antmicro-footprints:0402-cap, F.Cu at (314.3, 106.5)
- added C187: C_1u_0402, antmicro-footprints:0402-cap, F.Cu at (317.2, 104.5)
- added C188: C_100n_0402, antmicro-footprints:0402-cap, F.Cu at (302.4, 117.2)
- added C189: C_1u_0402, antmicro-footprints:0402-cap, F.Cu at (307.5, 153.7)
- added C190: C_1u_0402, antmicro-footprints:0402-cap, F.Cu at (306.3, 157.7)
- added C191: C_10u_0402, antmicro-footprints:0402-cap, F.Cu at (507.2, 73.2)
- added C192: C_22p_0402, antmicro-footprints:0402-cap, F.Cu at (511.1, 71.2)
- added C193: C_22p_0402, antmicro-footprints:0402-cap, F.Cu at (498.5, 86.0)
- added C194: C_10u_25V_0603, antmicro-footprints:0603-cap, F.Cu at (491.8, 78.8)
- added C195: C_100n_0201, antmicro-footprints:0201-res, F.Cu at (501.1, 87.3)
- added C196: C_100n_0201, antmicro-footprints:0201-res, F.Cu at (507.0, 80.8)
- added C197: C_100n_0201, antmicro-footprints:0201-res, F.Cu at (507.0, 79.1)
- added C198: C_100n_0201, antmicro-footprints:0201-res, F.Cu at (509.4, 78.8)
- added C199: C_10u_0402, antmicro-footprints:0402-cap, F.Cu at (495.6, 82.5)
- added C200: C_22p_0402, antmicro-footprints:0402-cap, F.Cu at (492.5, 87.0)
- added C201: C_10u_0402, antmicro-footprints:0402-cap, F.Cu at (495.4, 86.5)
- added C202: C_100n_0201, antmicro-footprints:0201-res, F.Cu at (512.8, 74.9)
- added C203: C_100n_0201, antmicro-footprints:0201-res, F.Cu at (511.8, 76.9)
- added C204: C_100n_0201, antmicro-footprints:0201-res, F.Cu at (509.7, 75.1)
- added C205: C_10u_0402, antmicro-footprints:0402-cap, F.Cu at (498.5, 80.1)
- added C206: C_22p_0402, antmicro-footprints:0402-cap, F.Cu at (504.1, 75.2)
- added C207: C_10u_0402, antmicro-footprints:0402-cap, F.Cu at (472.6, 88.0)
- added C208: C_100n_0201, antmicro-footprints:0201-res, F.Cu at (509.4, 77.1)
- added C209: C_100n_0201, antmicro-footprints:0201-res, F.Cu at (512.8, 73.1)
- added C210: C_100n_0201, antmicro-footprints:0201-res, F.Cu at (498.1, 87.9)
- added C211: C_100n_0201, antmicro-footprints:0201-res, F.Cu at (515.2, 73.1)
- added C212: C_100n_0201, antmicro-footprints:0201-res, F.Cu at (504.1, 81.6)
- added C213: C_10u_0402, antmicro-footprints:0402-cap, F.Cu at (495.6, 80.6)
- added C214: C_1u_0402, antmicro-footprints:0402-cap, F.Cu at (501.4, 83.7)
- added C215: C_100n_0201, antmicro-footprints:0201-res, F.Cu at (501.1, 85.5)
- added C216: C_100n_0201, antmicro-footprints:0201-res, F.Cu at (504.1, 83.3)
- added C217: C_22p_0402, antmicro-footprints:0402-cap, F.Cu at (424.3, 81.2)
- added C218: C_10u_0402, antmicro-footprints:0402-cap, F.Cu at (424.3, 77.2)
- added C219: C_10u_0402, antmicro-footprints:0402-cap, F.Cu at (392.4, 97.4)
- added C220: C_10u_0402, antmicro-footprints:0402-cap, F.Cu at (424.2, 71.2)
- added C221: C_22p_0402, antmicro-footprints:0402-cap, F.Cu at (424.2, 73.2)
- added C222: C_100n_0201, antmicro-footprints:0201-res, F.Cu at (413.7, 93.1)
- added C223: C_22p_0402, antmicro-footprints:0402-cap, F.Cu at (432.9, 71.2)
- added C224: C_100n_0201, antmicro-footprints:0201-res, F.Cu at (432.3, 77.1)
- added C225: C_100n_0201, antmicro-footprints:0201-res, F.Cu at (429.9, 77.1)
- added C226: C_100n_0201, antmicro-footprints:0201-res, F.Cu at (432.7, 73.1)
- added C227: C_100n_0201, antmicro-footprints:0201-res, F.Cu at (424.0, 83.1)
- added C228: C_22p_0402, antmicro-footprints:0402-cap, F.Cu at (386.6, 101.9)
- added C229: C_100n_0201, antmicro-footprints:0201-res, F.Cu at (406.8, 100.1)
- added C230: C_100n_0201, antmicro-footprints:0201-res, F.Cu at (406.3, 102.0)
- added C231: C_100n_0201, antmicro-footprints:0201-res, F.Cu at (370.4, 104.5)
- added C232: C_100n_0201, antmicro-footprints:0201-res, F.Cu at (409.7, 97.4)
- added C233: C_100n_0201, antmicro-footprints:0201-res, F.Cu at (403.9, 102.0)
- added C234: C_100n_0201, antmicro-footprints:0201-res, F.Cu at (426.9, 79.1)
- added C235: C_100n_0201, antmicro-footprints:0201-res, F.Cu at (423.2, 85.1)
- added C236: C_10u_0402, antmicro-footprints:0402-cap, F.Cu at (405.9, 89.8)
- added C237: C_100n_0201, antmicro-footprints:0201-res, F.Cu at (409.7, 99.1)
- added C238: C_10p_0402, antmicro-footprints:0402-cap, F.Cu at (404.1, 98.2)
- added C239: C_10u_0402, antmicro-footprints:0402-cap, F.Cu at (430.0, 71.2)
- added C240: C_10p_0402, antmicro-footprints:0402-cap, F.Cu at (424.3, 75.2)
- added C241: C_10p_0402, antmicro-footprints:0402-cap, F.Cu at (398.3, 101.4)
- added C242: C_100n_0201, antmicro-footprints:0201-res, F.Cu at (409.7, 95.6)
- added C243: C_10n_0402, antmicro-footprints:0402-cap, F.Cu at (430.1, 75.2)
- added C244: C_10p_0402, antmicro-footprints:0402-cap, F.Cu at (430.0, 73.2)
- added C245: C_10u_0402, antmicro-footprints:0402-cap, F.Cu at (394.7, 105.4)
- added C246: C_100n_0201, antmicro-footprints:0201-res, F.Cu at (420.3, 87.2)
- added C247: C_100n_0201, antmicro-footprints:0201-res, F.Cu at (435.2, 73.1)
- added C248: C_100n_0201, antmicro-footprints:0201-res, F.Cu at (416.6, 91.2)
- added C249: C_100n_0201, antmicro-footprints:0201-res, F.Cu at (420.3, 88.9)
- added C250: C_10u_0402, antmicro-footprints:0402-cap, F.Cu at (395.4, 103.4)
- added C251: C_100n_0201, antmicro-footprints:0201-res, F.Cu at (403.9, 103.8)
- added C252: C_100n_0201, antmicro-footprints:0201-res, F.Cu at (429.4, 79.1)
- added C253: C_100n_0201, antmicro-footprints:0201-res, F.Cu at (438.1, 71.1)
- added C254: C_100n_0201, antmicro-footprints:0201-res, F.Cu at (417.3, 89.2)
- added C255: C_100n_0201, antmicro-footprints:0201-res, F.Cu at (412.1, 95.6)
- added C256: C_100n_0201, antmicro-footprints:0201-res, F.Cu at (435.6, 71.1)
- added C257: C_100n_0201, antmicro-footprints:0201-res, F.Cu at (294.8, 97.0)
- added C258: C_47u_16V_1206, antmicro-footprints:1206-cap, F.Cu at (349.4, 71.9)
- added C259: C_100n_0402, antmicro-footprints:0402-cap, F.Cu at (293.3, 91.2)
- added C260: C_100n_0402, antmicro-footprints:0402-cap, F.Cu at (350.5, 74.6)
- added C261: C_100n_0402, antmicro-footprints:0402-cap, F.Cu at (354.2, 71.2)
- added C262: C_100n_0402, antmicro-footprints:0402-cap, F.Cu at (287.4, 91.2)
- added C263: C_100n_0402, antmicro-footprints:0402-cap, F.Cu at (287.4, 93.2)
- added C264: C_100n_0402, antmicro-footprints:0402-cap, F.Cu at (292.1, 97.1)
- added C265: C_100n_0402, antmicro-footprints:0402-cap, F.Cu at (354.2, 73.2)
- added C266: C_100n_0402, antmicro-footprints:0402-cap, F.Cu at (290.4, 91.2)
- added C267: C_100n_0402, antmicro-footprints:0402-cap, F.Cu at (284.5, 93.2)
- added C268: C_100n_0402, antmicro-footprints:0402-cap, F.Cu at (277.6, 97.4)
- added C269: C_100n_0402, antmicro-footprints:0402-cap, F.Cu at (293.3, 93.2)
- added C270: C_100n_0402, antmicro-footprints:0402-cap, F.Cu at (347.6, 76.6)
- added C271: C_100n_0402, antmicro-footprints:0402-cap, F.Cu at (284.5, 95.1)
- added C272: C_100n_0402, antmicro-footprints:0402-cap, F.Cu at (289.2, 97.1)
- added C273: C_100n_0402, antmicro-footprints:0402-cap, F.Cu at (283.4, 97.1)
- added C274: C_100n_0402, antmicro-footprints:0402-cap, F.Cu at (296.2, 91.2)
- added C275: C_10u_0402, antmicro-footprints:0402-cap, F.Cu at (397.6, 105.4)
- added C276: C_10u_0402, antmicro-footprints:0402-cap, F.Cu at (391.8, 105.4)
- added C277: C_100n_0201, antmicro-footprints:0201-res, F.Cu at (426.9, 80.8)
- added C278: C_100n_0201, antmicro-footprints:0201-res, F.Cu at (432.8, 74.9)
- added C279: C_1u_0402_16V, antmicro-footprints:0402-cap, F.Cu at (399.1, 174.2)
- added C280: C_22u_0805_25V, antmicro-footprints:0805-cap, F.Cu at (384.5, 173.9)
- added C281: C_1u_0402, antmicro-footprints:0402-cap, F.Cu at (411.3, 169.6)
- added C282: C_22u_0805_25V, antmicro-footprints:0805-cap, F.Cu at (378.4, 174.0)
- added C283: C_1u_0402, antmicro-footprints:0402-cap, F.Cu at (405.5, 170.6)
- added C284: C_22u_0603, antmicro-footprints:0603-cap, F.Cu at (406.9, 159.4)
- added C285: C_22u_0603, antmicro-footprints:0603-cap, F.Cu at (407.0, 156.9)
- added C286: C_22u_0603, antmicro-footprints:0603-cap, F.Cu at (405.6, 161.9)
- added C287: C_22u_0603, antmicro-footprints:0603-cap, F.Cu at (401.7, 165.1)
- added C288: C_22u_0603, antmicro-footprints:0603-cap, F.Cu at (414.1, 154.5)
- added C289: C_22u_0603, antmicro-footprints:0603-cap, F.Cu at (403.5, 154.5)
- added C290: C_1u_0402, antmicro-footprints:0402-cap, F.Cu at (429.3, 162.2)
- added C291: C_1u_0402, antmicro-footprints:0402-cap, F.Cu at (413.7, 159.2)
- added C292: C_100n_0402, antmicro-footprints:0402-cap, F.Cu at (423.5, 164.2)
- added C293: C_100n_0402, antmicro-footprints:0402-cap, F.Cu at (402.0, 173.3)
- added C294: C_100n_0402, antmicro-footprints:0402-cap, F.Cu at (408.4, 172.8)
- added C295: C_100n_0402, antmicro-footprints:0402-cap, F.Cu at (408.4, 168.9)
- added C296: C_22u_0805_25V, antmicro-footprints:0805-cap, F.Cu at (373.6, 174.0)
- added C297: C_470n_0402, antmicro-footprints:0402-cap, F.Cu at (417.2, 156.7)
- added C298: C_22u_0805_25V, antmicro-footprints:0805-cap, F.Cu at (399.1, 159.9)
- added C299: C_100n_0402, antmicro-footprints:0402-cap, F.Cu at (408.8, 164.9)
- added C300: C_10u_0402, antmicro-footprints:0402-cap, F.Cu at (416.6, 159.2)
- added C301: C_100n_0402, antmicro-footprints:0402-cap, F.Cu at (423.4, 168.6)
- added C302: C_1u_0402, antmicro-footprints:0402-cap, F.Cu at (417.1, 175.2)
- added C303: C_4u7_0402, antmicro-footprints:0402-cap, F.Cu at (414.8, 165.2)
- added C304: C_10u_0402, antmicro-footprints:0402-cap, F.Cu at (408.4, 170.8)
- added C305: C_1n_0402, antmicro-footprints:0402-res, F.Cu at (405.5, 172.5)
- added C306: C_1u_0402, antmicro-footprints:0402-cap, F.Cu at (398.3, 157.1)
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Connections:
- net /FPGA banks 12-15/SRAM.A0 renamed /DRAM + SRAM/SRAM.A0
- net /FPGA banks 12-15/SRAM.A1 renamed /DRAM + SRAM/SRAM.A1
- net /FPGA banks 12-15/SRAM.A10 renamed /DRAM + SRAM/SRAM.A10
- net /FPGA banks 12-15/SRAM.A11 renamed /DRAM + SRAM/SRAM.A11
- net /FPGA banks 12-15/SRAM.A12 renamed /DRAM + SRAM/SRAM.A12
- net /FPGA banks 12-15/SRAM.A13 renamed /DRAM + SRAM/SRAM.A13
- net /FPGA banks 12-15/SRAM.A14 renamed /DRAM + SRAM/SRAM.A14
- net /FPGA banks 12-15/SRAM.A15 renamed /DRAM + SRAM/SRAM.A15
- net /FPGA banks 12-15/SRAM.A16 renamed /DRAM + SRAM/SRAM.A16
- net /FPGA banks 12-15/SRAM.A17 renamed /DRAM + SRAM/SRAM.A17
- net /FPGA banks 12-15/SRAM.A18 renamed /DRAM + SRAM/SRAM.A18
- net /FPGA banks 12-15/SRAM.A19 renamed /DRAM + SRAM/SRAM.A19
- net /FPGA banks 12-15/SRAM.A2 renamed /DRAM + SRAM/SRAM.A2
- net /FPGA banks 12-15/SRAM.A3 renamed /DRAM + SRAM/SRAM.A3
- net /FPGA banks 12-15/SRAM.A4 renamed /DRAM + SRAM/SRAM.A4
- net /FPGA banks 12-15/SRAM.A5 renamed /DRAM + SRAM/SRAM.A5
- net /FPGA banks 12-15/SRAM.A6 renamed /DRAM + SRAM/SRAM.A6
- net /FPGA banks 12-15/SRAM.A7 renamed /DRAM + SRAM/SRAM.A7
- net /FPGA banks 12-15/SRAM.A8 renamed /DRAM + SRAM/SRAM.A8
- net /FPGA banks 12-15/SRAM.A9 renamed /DRAM + SRAM/SRAM.A9
- net /FPGA banks 12-15/SRAM.DQ0 renamed /DRAM + SRAM/SRAM.DQ0
- net /FPGA banks 12-15/SRAM.DQ1 renamed /DRAM + SRAM/SRAM.DQ1
- net /FPGA banks 12-15/SRAM.DQ2 renamed /DRAM + SRAM/SRAM.DQ2
- net /FPGA banks 12-15/SRAM.DQ3 renamed /DRAM + SRAM/SRAM.DQ3
- net /FPGA banks 12-15/SRAM.DQ4 renamed /DRAM + SRAM/SRAM.DQ4
- net /FPGA banks 12-15/SRAM.DQ5 renamed /DRAM + SRAM/SRAM.DQ5
- net /FPGA banks 12-15/SRAM.DQ6 renamed /DRAM + SRAM/SRAM.DQ6
- net /FPGA banks 12-15/SRAM.DQ7 renamed /DRAM + SRAM/SRAM.DQ7
- net /FPGA banks 33-34/DDR.A0 renamed /DRAM + SRAM/DDR.A0
- net /FPGA banks 33-34/DDR.A1 renamed /DRAM + SRAM/DDR.A1
- net /FPGA banks 33-34/DDR.A10 renamed /DRAM + SRAM/DDR.A10
- net /FPGA banks 33-34/DDR.A11 renamed /DRAM + SRAM/DDR.A11
- net /FPGA banks 33-34/DDR.A12 renamed /DRAM + SRAM/DDR.A12
- net /FPGA banks 33-34/DDR.A13 renamed /DRAM + SRAM/DDR.A13
- net /FPGA banks 33-34/DDR.A14 renamed /DRAM + SRAM/DDR.A14
- net /FPGA banks 33-34/DDR.A15 renamed /DRAM + SRAM/DDR.A15
- net /FPGA banks 33-34/DDR.A2 renamed /DRAM + SRAM/DDR.A2
- net /FPGA banks 33-34/DDR.A3 renamed /DRAM + SRAM/DDR.A3
- net /FPGA banks 33-34/DDR.A4 renamed /DRAM + SRAM/DDR.A4
- net /FPGA banks 33-34/DDR.A5 renamed /DRAM + SRAM/DDR.A5
- net /FPGA banks 33-34/DDR.A6 renamed /DRAM + SRAM/DDR.A6
- net /FPGA banks 33-34/DDR.A7 renamed /DRAM + SRAM/DDR.A7
- net /FPGA banks 33-34/DDR.A8 renamed /DRAM + SRAM/DDR.A8
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Routing:
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
Commit message: Re-annotate the schematic. Export changes to PCB
Parts:
- removed TP15, TP16, TP19: TP_SMD_0_75MM, antmicro-footprints:Testpoint_smd_0_75mm
- added C354: C_22n_0402, antmicro-footprints:0402-cap, F.Cu at (584.1, 107.3)
- added C355: C_10u_0402, antmicro-footprints:0402-cap, F.Cu at (567.1, 114.7)
- added C356: C_100n_0402, antmicro-footprints:0402-cap, F.Cu at (572.7, 105.3)
- added C357: C_22u_0603, antmicro-footprints:0603-cap, F.Cu at (560.9, 115.5)
- added C358: C_10u_0402, antmicro-footprints:0402-cap, F.Cu at (575.7, 119.8)
- added C359: C_22u_0603, antmicro-footprints:0603-cap, F.Cu at (547.6, 123.6)
- added C360: C_22u_0603, antmicro-footprints:0603-cap, F.Cu at (554.7, 121.2)
- added C361: C_10u_0402, antmicro-footprints:0402-cap, F.Cu at (569.5, 124.3)
- added C362: C_100n_0402, antmicro-footprints:0402-cap, F.Cu at (581.7, 115.3)
- added C363: C_22u_0603, antmicro-footprints:0603-cap, F.Cu at (558.6, 110.5)
- added C364: C_22p_0402, antmicro-footprints:0402-cap, F.Cu at (557.9, 122.4)
- added C365: C_22p_0402, antmicro-footprints:0402-cap, F.Cu at (531.1, 131.5)
- added C366: C_4u7_0402, antmicro-footprints:0402-cap, F.Cu at (524.6, 142.3)
- added C367: C_22p_0402, antmicro-footprints:0402-cap, F.Cu at (526.8, 138.2)
- added C368: C_100n_0402, antmicro-footprints:0402-cap, F.Cu at (531.1, 133.5)
- added C369: C_100n_0402, antmicro-footprints:0402-cap, F.Cu at (534.0, 131.5)
- added C370: C_100n_0402, antmicro-footprints:0402-cap, F.Cu at (534.0, 133.5)
- added C371: C_100n_0402, antmicro-footprints:0402-cap, F.Cu at (527.5, 140.2)
- added C372: C_100n_0402, antmicro-footprints:0402-cap, F.Cu at (518.7, 144.7)
- added C373: C_4u7_0402, antmicro-footprints:0402-cap, F.Cu at (529.7, 136.2)
- added C374: C_100n_0201, antmicro-footprints:0201-res, F.Cu at (604.2, 12.6)
- added C375: C_100n_0201, antmicro-footprints:0201-res, F.Cu at (607.1, 8.64)
- added D33: BZX84C5V1-TP, antmicro-footprints:SOT-23-3, F.Cu at (544.4, 117.4)
- added J13: USB4105-GF-A, antmicro-footprints:GCT_USB4105-GF-A, F.Cu at (448.5, 54.6)
- added J14: USB4105-GF-A, antmicro-footprints:GCT_USB4105-GF-A, F.Cu at (446.3, 45.1)
- added J15: 5-2337992-8, antmicro-footprints:5-2337992-8, F.Cu at (435.4, 68.4)
- added J16: 5-2337992-8, antmicro-footprints:5-2337992-8, F.Cu at (454.9, 68.4)
- added J17: 685119134923_alt_symbol, antmicro-footprints:HDMI_A_Female_685119134923, F.Cu at (479.9, 75.2)
- added J18: ASP-184329-01_mounting_holes_FMCPinout, antmicro-footprints:ASP-184329-01_mounting_holes, F.Cu at (160.5, 105.8)
- added Q16: BSS138PW, antmicro-footprints:SC70-3, F.Cu at (546.0, 59.4)
- added Q17: BSS138PW, antmicro-footprints:SC70-3, F.Cu at (444.9, 59.7)
- added R310: R_0R_0402, antmicro-footprints:0402-res, F.Cu at (583.5, 109.3)
- added R311: R_0R_0402, antmicro-footprints:0402-res, F.Cu at (578.8, 111.3)
- added R312: R_0R_0402, antmicro-footprints:0402-res, F.Cu at (570.0, 114.3)
- added R313: R_0R_0402, antmicro-footprints:0402-res, F.Cu at (570.0, 112.4)
- added R314: R_0R_0402, antmicro-footprints:0402-res, F.Cu at (575.9, 113.8)
- added R315: R_0R_0402, antmicro-footprints:0402-res, F.Cu at (575.6, 105.3)
- added R316: R_0R_0402, antmicro-footprints:0402-res, F.Cu at (560.8, 119.7)
- added R317: R_0R_0402, antmicro-footprints:0402-res, F.Cu at (578.8, 113.3)
- added R318: R_47k_0402, antmicro-footprints:0402-res, F.Cu at (578.3, 107.3)
- added R319: R_0R_0402, antmicro-footprints:0402-res, F.Cu at (560.8, 117.7)
- added R320: R_0R_0402, antmicro-footprints:0402-res, F.Cu at (581.7, 113.3)
- added R321: R_47k_0402, antmicro-footprints:0402-res, F.Cu at (569.5, 120.3)
- added R322: R_47k_0402, antmicro-footprints:0402-res, F.Cu at (560.2, 125.7)
- added R323: R_10k_0402, antmicro-footprints:0402-res, F.Cu at (569.5, 126.3)
- added R324: R_10k_0402, antmicro-footprints:0402-res, F.Cu at (575.9, 111.8)
- added R325: R_4k7_0402, antmicro-footprints:0402-res, F.Cu at (581.2, 107.3)
- added R326: R_0R_0603_HPWR, antmicro-footprints:0603-res, F.Cu at (565.9, 108.1)
- added R327: R_10k_0402, antmicro-footprints:0402-res, F.Cu at (574.8, 109.8)
- added R328: R_0R_0402, antmicro-footprints:0402-res, F.Cu at (569.9, 118.3)
- added R329: R_0R_0402, antmicro-footprints:0402-res, F.Cu at (575.9, 115.8)
- added R330: R_0R_0603_HPWR, antmicro-footprints:0603-res, F.Cu at (544.0, 123.6)
- added R331: R_80k6_0402, antmicro-footprints:0402-res, F.Cu at (567.1, 112.8)
- added R332: R_205k_0402, antmicro-footprints:0402-res, F.Cu at (577.7, 109.3)
- added R333: R_0R_0603_HPWR, antmicro-footprints:0603-res, F.Cu at (558.8, 108.1)
- added R334: R_100R_0402, antmicro-footprints:0402-res, F.Cu at (524.6, 140.3)
- added R335: R_22R_0402, antmicro-footprints:0402-res, F.Cu at (521.6, 144.7)
- added R336: R_22R_0402, antmicro-footprints:0402-res, F.Cu at (526.8, 136.2)
- added R337: R_22R_0402, antmicro-footprints:0402-res, F.Cu at (518.7, 146.7)
- added R338: R_1k_0402, antmicro-footprints:0402-res, F.Cu at (518.7, 83.4)
- added R339: R_80R6_0402, antmicro-footprints:0402-res, F.Cu at (604.5, 8.76)
- added R340: R_80R6_0402, antmicro-footprints:0402-res, F.Cu at (604.5, 10.7)
- added TP6: TP_SMD_0_75MM, antmicro-footprints:Testpoint_smd_0_75mm, F.Cu at (567.1, 126.6)
- added TP7: TP_SMD_0_75MM, antmicro-footprints:Testpoint_smd_0_75mm, F.Cu at (565.4, 126.6)
- added TP8: TP_SMD_0_75MM, antmicro-footprints:Testpoint_smd_0_75mm, F.Cu at (555.9, 108.2)
- added U37: MP8869S, antmicro-footprints:MPS_QFN-14_MP8869S, F.Cu at (540.2, 107.4)
- added U38: TPS7A20185PDQNR, antmicro-footprints:XDFN4, F.Cu at (569.6, 108.1)
- added U39: NCP51400MNTXG, antmicro-footprints:DFN-10-1EP_3x3mm, F.Cu at (549.7, 112.0)
- added U40: XC6230H001ER-G, antmicro-footprints:Torex_USP-6C, F.Cu at (549.7, 116.2)
- added U41: REF3012AIDBZT, antmicro-footprints:SOT-23-3, F.Cu at (539.7, 118.2)
- added U42: CDCE906PWR, antmicro-footprints:TSSOP-20_W4.4mm, F.Cu at (521.3, 134.9)
- added Y5: ABM8G-12.000MHZ-18-D2Y-T, antmicro-footprints:KX-7, F.Cu at (520.6, 141.5)
- added Y6: AX3DCF1-200.0000, antmicro-footprints:AX3DAF1, F.Cu at (527.5, 132.6)
- C1: value C_47u_0603 -> C_330u_KEMET_B; footprint antmicro-footprints:0603-cap -> antmicro-footprints:KEMET_B
- C10, C11, C12, C14, C16, C23: value C_4u7_0402 -> C_100n_0201; footprint antmicro-footprints:0402-cap -> antmicro-footprints:0201-res
- C105, C106, C107, C108, C109, C166, C46, C49: value C_100n_0201 -> C_47u_0603; footprint antmicro-footprints:0201-res -> antmicro-footprints:0603-cap
- C110, C160, C161, C162, C163, C34, C349, C45, C48, C66, C80, C86: value C_100n_0201 -> C_4u7_0402; footprint antmicro-footprints:0201-res -> antmicro-footprints:0402-cap
- C112, C120, C125, C130, C133: value C_100n_0201 -> C_330u_KEMET_B; footprint antmicro-footprints:0201-res -> antmicro-footprints:KEMET_B
- C13, C15, C17, C18, C19, C20, C21, C24, C53, C64: value C_47u_0603 -> C_100n_0201; footprint antmicro-footprints:0603-cap -> antmicro-footprints:0201-res
- C164, C203, C204, C209, C210, C212, C336, C337, C338, C339, C343, C347: value C_100n_0201 -> C_100n_0402; footprint antmicro-footprints:0201-res -> antmicro-footprints:0402-cap
- C165: value C_100n_0201 -> C_2n2_0402; footprint antmicro-footprints:0201-res -> antmicro-footprints:0402-cap
- C167: value C_100n_0402 -> C_47u_0603; footprint antmicro-footprints:0402-cap -> antmicro-footprints:0603-cap
- C168: value C_1u_0603_25V -> C_4u7_0402; footprint antmicro-footprints:0603-cap -> antmicro-footprints:0402-cap
- C169: value C_1u_0402 -> C_4u7_0402
- C170, C187, C281, C283, C290, C291, C56: value C_1u_0402 -> C_100n_0201; footprint antmicro-footprints:0402-cap -> antmicro-footprints:0201-res
- C171: value C_100n_0805_100V -> C_100n_0201; footprint antmicro-footprints:0805-cap -> antmicro-footprints:0201-res
- C172, C173, C174, C176: value C_22u_2220_100V -> C_100n_0201; footprint antmicro-footprints:2220-cap -> antmicro-footprints:0201-res
- C175: value C_100n_0402_50V -> C_100n_0201; footprint antmicro-footprints:0402-cap -> antmicro-footprints:0201-res
- C177, C178, C179: value C_47u_16V_1206 -> C_100n_0201; footprint antmicro-footprints:1206-cap -> antmicro-footprints:0201-res
- C180, C188, C271, C274, C292, C293: value C_100n_0402 -> C_10u_0402
- C181, C182, C186, C259, C260, C261, C262, C264, C265, C266, C267, C268, C269, C270, C272, C294, C295, C63: value C_100n_0402 -> C_100n_0201; footprint antmicro-footprints:0402-cap -> antmicro-footprints:0201-res
- C183, C184, C185: value C_1u_0603_25V -> C_100n_0201; footprint antmicro-footprints:0603-cap -> antmicro-footprints:0201-res
- C189: value C_1u_0402 -> C_10u_0402
- C190, C302, C306, C308: value C_1u_0402 -> C_100n_0402
- C191, C207: value C_10u_0402 -> C_1u_0603_25V; footprint antmicro-footprints:0402-cap -> antmicro-footprints:0603-cap
- C192, C193, C217: value C_22p_0402 -> C_1u_0402
- C194: value C_10u_25V_0603 -> C_100n_0805_100V; footprint antmicro-footprints:0603-cap -> antmicro-footprints:0805-cap
- C195, C196, C197: value C_100n_0201 -> C_22u_2220_100V; footprint antmicro-footprints:0201-res -> antmicro-footprints:2220-cap
- C198: value C_100n_0201 -> C_100n_0402_50V; footprint antmicro-footprints:0201-res -> antmicro-footprints:0402-cap
- C199: value C_10u_0402 -> C_22u_2220_100V; footprint antmicro-footprints:0402-cap -> antmicro-footprints:2220-cap
- C200: value C_22p_0402 -> C_47u_16V_1206; footprint antmicro-footprints:0402-cap -> antmicro-footprints:1206-cap
- C201: value C_10u_0402 -> C_47u_16V_1206; footprint antmicro-footprints:0402-cap -> antmicro-footprints:1206-cap
- C202: value C_100n_0201 -> C_47u_16V_1206; footprint antmicro-footprints:0201-res -> antmicro-footprints:1206-cap
- C205, C300, C304, C309: value C_10u_0402 -> C_100n_0402
- C206: value C_22p_0402 -> C_1u_0603_25V; footprint antmicro-footprints:0402-cap -> antmicro-footprints:0603-cap
- C208: value C_100n_0201 -> C_1u_0603_25V; footprint antmicro-footprints:0201-res -> antmicro-footprints:0603-cap
- C211, C215, C216, C334, C335, C346, C348: value C_100n_0201 -> C_1u_0402; footprint antmicro-footprints:0201-res -> antmicro-footprints:0402-cap
- C213: value C_10u_0402 -> C_1u_0402
- C218: value C_10u_0402 -> C_10u_25V_0603; footprint antmicro-footprints:0402-cap -> antmicro-footprints:0603-cap
- C22, C52: value C_47u_0603 -> C_4u7_0402; footprint antmicro-footprints:0603-cap -> antmicro-footprints:0402-cap
- C220: value C_10u_0402 -> C_22p_0402
- C221: value C_22p_0402 -> C_10u_0402
- C222: value C_100n_0201 -> C_10u_25V_0603; footprint antmicro-footprints:0201-res -> antmicro-footprints:0603-cap
- C225, C229, C234, C242, C253, C254, C255, C340, C344: value C_100n_0201 -> C_10u_0402; footprint antmicro-footprints:0201-res -> antmicro-footprints:0402-cap
- C235, C252, C256: value C_100n_0201 -> C_22p_0402; footprint antmicro-footprints:0201-res -> antmicro-footprints:0402-cap
- C238, C240, C241, C244: value C_10p_0402 -> C_100n_0201; footprint antmicro-footprints:0402-cap -> antmicro-footprints:0201-res
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Connections:
- C1 pad 1: +3V3 -> +1V0
- C10 pad 1: +1V0 -> +3V3
- C100 pad 1: +1V0 -> +1V8
- C102 pad 1: +1V8 -> +1V35
- C103 pad 1: +1V0 -> +1V2_MGTAVCC
- C104 pad 1: VCCO_17 -> +1V2_MGTAVCC
- C105 pad 1: +1V35 -> VCCO_17
- C106 pad 1: +1V8 -> VCCO_18
- C108 pad 1: +1V0 -> +1V8
- C109 pad 1: VCCO_17 -> +1V35
- C11 pad 1: +1V0 -> +3V3
- C110 pad 1: VCCO_18 -> +1V8
- C111 pad 1: +1V8 -> +1V2_MGTAVCC
- C112 pad 1: +1V8 -> +1V0
- C113 pad 1: +1V35 -> +1V0
- C114 pad 1: +1V8 -> +1V0
- C115 pad 1: +1V8 -> +1V2_MGTAVCC
- C117 pad 1: VCCO_17 -> +1V0
- C118 pad 1: VCCO_18 -> +1V8
- C119 pad 1: +1V8 -> +1V2_MGTAVCC
- C12 pad 1: +1V0 -> +3V3
- C120 pad 1: +1V8 -> +1V0
- C121 pad 1: +1V35 -> +1V0
- C122 pad 1: VCCO_17 -> +1V0
- C123 pad 1: VCCO_18 -> +1V8
- C124 pad 1: +1V8 -> +1V2_MGTAVCC
- C125 pad 1: +1V8 -> +1V0
- C126 pad 1: +1V35 -> +1V0
- C127 pad 1: VCCO_17 -> +1V0
- C128 pad 1: VCCO_18 -> +1V0
- C129 pad 1: +1V8 -> +1V0
- C13 pad 1: +1V8 -> +3V3
- C130 pad 1: +1V8 -> +1V0
- C131 pad 1: +1V35 -> +1V0
- C132 pad 1: VCCO_17 -> +1V0
- C133 pad 1: VCCO_18 -> +1V0
- C134 pad 1: +1V8 -> +1V0
- C135 pad 1: +1V8 -> +1V0
- C136 pad 1: +1V35 -> +1V0
- C137 pad 1: VCCO_17 -> +1V0
- C138 pad 1: VCCO_18 -> +1V0
- C139 pad 1: +1V8 -> +1V0
- C14 pad 1: +1V0 -> VCCO_15
- C140 pad 1: +1V8 -> +1V0
- C141 pad 1: +1V35 -> +1V0
- C142 pad 1: +1V0 -> +1V2_MGTAVTT
- C143 pad 1: +1V0 -> +1V2_MGTAVTT
- C144 pad 1: +1V0 -> +1V2_MGTAVTT
- C145 pad 1: +1V0 -> +1V2_MGTAVTT
- C146 pad 1: +1V0 -> +1V2_MGTAVTT
- C147 pad 1: +1V0 -> +1V2_MGTAVTT
- C148 pad 1: +1V0 -> +1V2_MGTAVTT
- C149 pad 1: +1V0 -> +1V2_MGTAVTT
- C15 pad 1: +1V8 -> VCCO_16
- C150 pad 1: +1V0 -> +1V2_MGTAVTT
- C151 pad 1: +1V0 -> +1V2_MGTAVTT
- C152 pad 1: +1V0 -> +1V2_MGTAVTT
- C153 pad 1: +1V0 -> +1V2_MGTAVTT
- C154 pad 1: +1V0 -> +1V2_MGTAVTT
- C155 pad 1: +1V0 -> +1V2_MGTAVTT
- C156 pad 1: +1V0 -> +1V2_MGTAVTT
- C157 pad 1: +1V0 -> +1V2_MGTAVTT
- C158 pad 1: +1V0 -> +1V2_MGTAVTT
- C159 pad 1: +1V0 -> +1V2_MGTAVTT
- C16 pad 1: +1V0 -> +3V3
- C160 pad 1: +1V0 -> +1V2_MGTAVTT
- C161 pad 1: +1V0 -> +1V2_MGTAVTT
- C162 pad 1: MGTAVTT -> +1V2_MGTAVTT
- C163 pad 1: MGTAVTT -> +1V2_MGTAVTT
- C164 pad 1: MGTAVTT -> +3V3
- C165 pad 1: +0V675_VREF -> Net-(C165-Pad1)
- C165 pad 2: EP -> Net-(C165-Pad2)
- C166 pad 1: +0V675_VREF -> +1V35
- C166 pad 2: EP -> +0V675_VTT
- C167 pad 1: /Power supply/DC_IN -> +0V675_VTT
- C168 pad 1: /Power supply/PD_VBUS -> +1V35
- C168 pad 2: EP -> +0V675_VTT
- C169 pad 1: /Power supply/VREG_1V2 -> +0V675_VTT
- C17 pad 1: +1V8 -> +3V3
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Routing:
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
Commit message: Start creating PCB technology mock
Parts:
- removed C1, C112, C120, C125, C130, C133: C_330u_KEMET_B, antmicro-footprints:KEMET_B
- removed C10, C100, C101, C102, C103, C104, C11, C111, C113, C114, C115, C116, C117, C118, C119, C12, C121, C122, C123, C124, C126, C127, C128, C129, C13, C131, C132, C134, C135, C136, C137, C138, C139, C14, C140, C141, C142, C143, C144, C145, C146, C147, C148, C149, C15, C150, C151, C152, C153, C154, C155, C156, C157, C158, C159, C16, C17, C170, C171, C172, C173, C174, C175, C176, C177, C178, C179, C18, C181, C182, C183, C184, C185, C186, C187, C19, C20, C21, C224, C226, C227, C23, C230, C231, C232, C233, C237, C238, C239, C24, C240, C241, C244, C245, C246, C247, C248, C249, C25, C250, C251, C257, C259, C26, C260, C261, C262, C264, C265, C266, C267, C268, C269, C27, C270, C272, C277, C281, C282, C283, C284, C286, C287, C288, C289, C29, C290, C291, C294, C295, C296, C30, C31, C32, C33, C35, C36, C37, C374, C375, C38, C39, C40, C41, C42, C43, C44, C47, C53, C55, C56, C58, C59, C60, C61, C62, C63, C64, C65, C67, C68, C69, C70, C71, C72, C73, C74, C75, C76, C77, C78, C79, C81, C82, C83, C84, C85, C87, C88, C89, C90, C91, C92, C93, C94, C95, C96, C97, C98, C99: C_100n_0201, antmicro-footprints:0201-res
- removed C105, C106, C107, C108, C109, C166, C167, C2, C3, C4, C46, C49, C5, C51, C54, C6, C7: C_47u_0603, antmicro-footprints:0603-cap
- removed C110, C160, C161, C162, C163, C168, C169, C22, C28, C34, C349, C366, C373, C45, C48, C50, C52, C57, C66, C8, C80, C86, C9: C_4u7_0402, antmicro-footprints:0402-cap
- removed C164, C190, C203, C204, C205, C209, C210, C212, C298, C299, C300, C301, C302, C303, C304, C305, C306, C307, C308, C309, C310, C311, C312, C313, C336, C337, C338, C339, C343, C347, C351, C356, C362, C368, C369, C370, C371, C372: C_100n_0402, antmicro-footprints:0402-cap
- removed C165: C_2n2_0402, antmicro-footprints:0402-cap
- removed C180, C188, C189, C219, C221, C225, C229, C234, C236, C242, C253, C254, C255, C271, C274, C280, C285, C292, C293, C340, C344, C353, C355, C358, C361: C_10u_0402, antmicro-footprints:0402-cap
- removed C191, C206, C207, C208: C_1u_0603_25V, antmicro-footprints:0603-cap
- removed C192, C193, C211, C213, C214, C215, C216, C217, C243, C316, C318, C321, C334, C335, C346, C348, C352: C_1u_0402, antmicro-footprints:0402-cap
- removed C194: C_100n_0805_100V, antmicro-footprints:0805-cap
- removed C195, C196, C197, C199: C_22u_2220_100V, antmicro-footprints:2220-cap
- removed C198: C_100n_0402_50V, antmicro-footprints:0402-cap
- removed C200, C201, C202, C297: C_47u_16V_1206, antmicro-footprints:1206-cap
- removed C218, C222: C_10u_25V_0603, antmicro-footprints:0603-cap
- removed C220, C223, C228, C235, C252, C256, C258, C263, C364, C365, C367: C_22p_0402, antmicro-footprints:0402-cap
- removed C273, C275, C276, C279: C_10p_0402, antmicro-footprints:0402-cap
- removed C278: C_10n_0402, antmicro-footprints:0402-cap
- removed C314: C_1u_0402_16V, antmicro-footprints:0402-cap
- removed C315, C317, C319, C320, C341, C345: C_22u_0805_25V, antmicro-footprints:0805-cap
- removed C322, C323, C324, C325, C326, C327, C328, C329, C330, C331, C332, C333, C357, C359, C360, C363: C_22u_0603, antmicro-footprints:0603-cap
- removed C342: C_470n_0402, antmicro-footprints:0402-cap
- removed C350: C_1n_0402, antmicro-footprints:0402-res
- removed C354: C_22n_0402, antmicro-footprints:0402-cap
- removed D1, D12, D18, D19, D2, D20, D21, D22, D23, D26, D27, D28, D29: KP-1608CGCK, antmicro-footprints:LED_0603
- removed D10: PTVS58VS1UR,115, antmicro-footprints:SOD-123F
- removed D11, D25: KP-1608QBC-D, antmicro-footprints:LED_0603
- removed D13, D24, D9: KP-1608EC, antmicro-footprints:LED_0603
- removed D14, D8: ESDA25P35-1U1M, antmicro-footprints:0603-diode
- removed D15, D16, D17, D32: PMEG3050EP,115, antmicro-footprints:Nexperia_SOD128
- removed D3: SMF4L15CA, antmicro-footprints:SOD-123FL
- removed D30: BAT54-02V-V-G, antmicro-footprints:SOD-523
- removed D31: RB521S30T1G, antmicro-footprints:SOD-523
- removed D33: BZX84C5V1-TP, antmicro-footprints:SOT-23-3
- removed D4, D5, D6, D7: CD-MMBL110S, antmicro-footprints:DFN3538
- removed FB1, FB2, FB3, FB4: BLM21PG221SN1D, antmicro-footprints:0805-res
- removed FB10, FB7, FB8, FB9: BLM18PG121SN1D, antmicro-footprints:0603-res
- removed FB11: BLM15PD121SN1D, antmicro-footprints:0402-res
- removed FB5, FB6: BLM18AG601SN1D, antmicro-footprints:0603
- removed IC1: ACPL-217-500E, antmicro-footprints:SOIC127P700X242-4N
- removed J1: 878321412, antmicro-footprints:PinHeader_2x7_P2mm_SMD_no_locator
- removed J10: 61232020621, antmicro-footprints:61232020621
- removed J12: 614004184726, antmicro-footprints:614004184726
- removed J13, J14: USB4105-GF-A, antmicro-footprints:GCT_USB4105-GF-A
- removed J15, J16: 5-2337992-8, antmicro-footprints:5-2337992-8
- removed J17: 685119134923_alt_symbol, antmicro-footprints:HDMI_A_Female_685119134923
- removed J2: DC_SOCKET, antmicro-footprints:DC_SOCKET
- removed J4, J7, J8: SM04B-SRSS-TB-LF-SN, antmicro-footprints:SM04B-SRSS-TB-LF-SN
- removed J5, J6: PMOD-2x6-artyA7_spacing, antmicro-footprints:pmod_pin_array_6x2
- removed L1: SRP6050CA-1R5M, antmicro-footprints:Bourns-SRP6050CA
- removed Q1, Q2: BSS138W-7-F, antmicro-footprints:SOT-323
- removed Q10, Q11, Q13, Q14, Q15, Q16, Q17, Q8, Q9: BSS138PW, antmicro-footprints:SC70-3
- removed Q12: IRLML6344TRPBF, antmicro-footprints:SOT-23-3
- removed Q3, Q4, Q5, Q6, Q7: SI7613DN-T1-GE3, antmicro-footprints:Vishay_PowerPAK_1212-8_Single
- removed R1, R112, R113, R114, R115, R116, R117, R118, R119, R120, R121, R122, R123, R124, R125, R126, R127, R134, R135, R136, R137, R138, R139, R142, R143, R144, R145, R146, R147, R334, R54, R70, R71, R72, R73, R96, R97, R98: R_100R_0402, antmicro-footprints:0402-res
- removed R10, R9: R_330R_0603, antmicro-footprints:0603-res
- removed R100, R101, R102, R103, R104, R105, R165, R180, R181, R186, R187, R188, R189, R243, R254, R255, R256, R257, R258, R259, R260, R261, R279, R280, R281, R282, R295, R296, R297, R298, R299, R300, R301, R302, R303, R304, R305, R306, R307, R308, R309, R310, R311, R312, R313, R314, R315, R316, R317, R319, R320, R328, R329, R49, R60, R62, R74, R75, R76, R77, R78, R79, R80, R81, R82, R83, R84, R85, R99: R_0R_0402, antmicro-footprints:0402-res
- removed R106, R107, R108, R109, R110, R111, R128, R129, R130, R131, R150, R151, R152, R153, R198, R240, R338, R45, R56, R57, R58, R59, R61, R63: R_1k_0402, antmicro-footprints:0402-res
- removed R11, R140, R141, R148, R149, R156, R157, R158, R159, R190, R191, R192, R194, R195, R197, R199, R2, R200, R201, R202, R203, R204, R205, R206, R207, R208, R219, R220, R221, R222, R223, R224, R239, R265, R266, R3, R323, R324, R327, R34, R4, R5, R6, R64, R65, R66, R67, R68, R69, R7, R8, R86, R87, R88, R89, R90, R91, R92, R93, R94, R95: R_10k_0402, antmicro-footprints:0402-res
- removed R12, R13, R14, R15, R16, R17, R18, R19, R20, R21, R22, R23, R24, R25, R26, R27, R28, R29, R30, R31, R33, R36, R37, R38, R39, R40, R41, R42, R43, R44: R_40R2_0201, antmicro-footprints:0201-res
- removed R132, R133: 4x10k_0201_array, antmicro-footprints:EXB18V
- removed R154, R155, R161, R162, R163, R164, R173, R174, R176, R177, R178, R179, R182, R183, R184, R185, R269, R270, R271, R272, R273, R274, R275, R276: R_33R_0402, antmicro-footprints:0402-res
- removed R160, R244, R248: R_12k_0402, antmicro-footprints:0402-res
- removed R166, R175, R283, R284, R293, R294, R318, R321, R322: R_47k_0402, antmicro-footprints:0402-res
- removed R167, R168, R171, R172: R_1k5_0402, antmicro-footprints:0402-res
- removed R169, R170: R_15k_0402, antmicro-footprints:0402-res
- removed R193, R196, R267, R268, R325: R_4k7_0402, antmicro-footprints:0402-res
- removed R209, R210, R211, R212, R213, R214, R215, R216, R217, R218, R225, R226, R227, R228, R229, R230: R_2k2_0402, antmicro-footprints:0402-res
- removed R231, R232, R233, R234, R235, R236, R237, R238: R_10R_1%_0402, antmicro-footprints:0402-res
- removed R241, R242: R_1M0_0402, antmicro-footprints:0402-res
- removed R245, R247, R249, R250: R_49R9_0402, antmicro-footprints:0402-res
- removed R246, R253: R_10R_0603, antmicro-footprints:0603-res
- removed R251, R252, R262, R263: R_220R_0603, antmicro-footprints:0603-res
- removed R264, R50: R_100k_0402, antmicro-footprints:0402-res
- removed R277: R_510k_0402, antmicro-footprints:0402-res
- removed R278: R_330k_0402, antmicro-footprints:0402-res
- removed R285, R286, R287, R288, R289, R290, R291, R292, R326, R330, R333: R_0R_0603_HPWR, antmicro-footprints:0603-res
- removed R32: R_100R_0201, antmicro-footprints:0201-res
- removed R331: R_80k6_0402, antmicro-footprints:0402-res
- removed R332: R_205k_0402, antmicro-footprints:0402-res
- removed R335, R336, R337: R_22R_0402, antmicro-footprints:0402-res
- removed R339, R340: R_80R6_0402, antmicro-footprints:0402-res
- removed R35: R_240R_1%_0402, antmicro-footprints:0402-res
- removed R46: R_32k4_0402, antmicro-footprints:0402-res
- removed R47: R_1k3_0402, antmicro-footprints:0402-res
- removed R48: R_49k9_0402, antmicro-footprints:0402-res
- removed R51: R_22k_0402, antmicro-footprints:0402-res
- removed R52: R_63R4_0603, antmicro-footprints:0603-res
- removed R53: R_1k2_0402, antmicro-footprints:0402-res
- removed R55: R_24k9_0402, antmicro-footprints:0402-res
- removed S1: B3U-1000P, antmicro-footprints:Switch_Tactile_SMD_B3U-1000P
- removed S2, S3, S4, S5: KMR2, antmicro-footprints:SW_SPST_4.2x2.8
- removed S6: 1-1825027-1, antmicro-footprints:TE_1-1825027-1
- removed SW1: CVS-03B, antmicro-footprints:SW_DIP_SPSTx03_Slide_Copal_CVS-03xB_W5.9mm_P1mm
- removed SW2: CVS-08TB, antmicro-footprints:SW_DIP_SPSTx08_Slide_Copal_CVS-08xB_W5.9mm_P1mm
- removed TP1, TP2, TP3, TP4, TP5, TP6, TP7, TP8: TP_SMD_0_75MM, antmicro-footprints:Testpoint_smd_0_75mm
- removed U10, U11, U9: LTC4412IS6, antmicro-footprints:SOT-23-6
- removed U12, U13, U14: MT25QL256ABA1EW7-0SIT, antmicro-footprints:WDFN-8-1EP_6x5mm_P1.27mm_EP3.4x4mm
- removed U15: TPS7B8133DRVR, antmicro-footprints:WSON6_TI_2x2mm
- removed U16, U17, U2, U21, U28, U29: TPD4E05U06QDQARQ1, antmicro-footprints:USON-10_2.5x1.0mm_P0.5mm
- removed U18: SN74HC595D, antmicro-footprints:SOIC-16_W3.90mm
- removed U19: MAX3421EETJ+, antmicro-footprints:QFN-32-1EP_5x5mm
- removed U20: FT4232H-56Q, antmicro-footprints:QFN-56-1EP_8x8mm_P0.5mm_EP5.5.9x5.9mm
- removed U22, U23, U24: TXU0304BQAR, antmicro-footprints:DHVQFN14
- removed U25: TUSB1106RSVR, antmicro-footprints:Texas_16-UFQFN
- removed U26: LAN8720A-CP-TR-ABC, antmicro-footprints:QFN-24-1EP_4x4mm_P0.5mm_EP2.6x2.6mm
- removed U27: KSZ9131RNXC, antmicro-footprints:QFN-48-Microchip-QFN77-48LD-PL-2
- removed U3: MAX1617AMEE+T, antmicro-footprints:QSOP-16_3.9x4.9mm_P0.635mm
- removed U30: NCP718ASN500T1G, antmicro-footprints:SOT-23-5
- removed U31, U32: MPM54304GMN, antmicro-footprints:MPS_LGA-33
- removed U33: MAX16150AUT+T, antmicro-footprints:SOT-23-6
- removed U34: NCP451AFCT2G, antmicro-footprints:Onsemi_WLCSP6_1.40x0.90
- removed U35: SN74LVC1G125DBVR, antmicro-footprints:SOT-753
- removed U36: LM3880, antmicro-footprints:SOT-23-6
- removed U37: MP8869S, antmicro-footprints:MPS_QFN-14_MP8869S
- removed U38: TPS7A20185PDQNR, antmicro-footprints:XDFN4
- removed U39: NCP51400MNTXG, antmicro-footprints:DFN-10-1EP_3x3mm
- removed U40: XC6230H001ER-G, antmicro-footprints:Torex_USP-6C
- removed U41: REF3012AIDBZT, antmicro-footprints:SOT-23-3
- removed U42: CDCE906PWR, antmicro-footprints:TSSOP-20_W4.4mm
- removed U6: STUSB4500QTR, antmicro-footprints:QFN50P400X400X90-25N
- removed U7: TPS2372-3RGWR, antmicro-footprints:Texas_RGW0020B
- removed U8: ULS-12/5-D48N-C, antmicro-footprints:ULS-12_5-D48N-C
- removed Y1, Y2, Y5: ABM8G-12.000MHZ-18-D2Y-T, antmicro-footprints:KX-7
- removed Y3, Y4: ABM8G-25.000MHZ-18-D2Y-T, antmicro-footprints:KX-7
- removed Y6: AX3DCF1-200.0000, antmicro-footprints:AX3DAF1
- added REF**: mounting-hole-4.2mm-NPTH, antmicro-footprints:mounting-hole-4.2mm-NPTH, F.Cu at (153.3, 186.7)
- added REF**: mounting-hole-4.2mm-NPTH, antmicro-footprints:mounting-hole-4.2mm-NPTH, F.Cu at (153.3, 73.3)
- added REF**: mounting-hole-4.2mm-NPTH, antmicro-footprints:mounting-hole-4.2mm-NPTH, F.Cu at (266.7, 73.3)
- added REF**: mounting-hole-4.2mm-NPTH, antmicro-footprints:mounting-hole-4.2mm-NPTH, F.Cu at (266.7, 186.7)
- moved U5 435.3 mm to (198.5, 155.3), turned to 180 degrees
- moved U4 377.3 mm to (240.1, 135.2)
- moved J3 356.9 mm to (210.4, 186.1)
- moved J11 346.5 mm to (222.9, 87.0)
- moved J9 282.6 mm to (255.8, 104.0), turned to 90 degrees
- moved J18 7.31 mm to (160.2, 113.1)
Routing:
- net EP: track 123.7 -> 199.5 mm, vias 175 -> 334
- net +1V2_MGTAVTT: track 13.4 -> 0.71 mm
- net /FMC+ HSPC/GTX115.REFCLK1_P: track 0.71 -> 9.41 mm
- net /FMC+ HSPC/GTX115.REFCLK1_N: track 0.71 -> 9.02 mm
- net /FPGA MGT Interface/GTX118.RX3_P: track 0.71 -> 8.97 mm
- net /FPGA MGT Interface/GTX118.REFCLK1_P: track 0.71 -> 8.97 mm
- net /FPGA MGT Interface/GTX118.REFCLK0_P: track 0.71 -> 8.97 mm
- net /FPGA MGT Interface/GTX117.REFCLK1_P: track 0.71 -> 8.97 mm
- net /FPGA MGT Interface/GTX117.REFCLK0_P: track 0.71 -> 8.97 mm
- net /FMC+ HSPC/GTX116.REFCLK1_P: track 0.71 -> 8.97 mm
- net /FMC+ HSPC/GTX116.REFCLK0_P: track 0.71 -> 8.97 mm
- net /FMC+ HSPC/GTX115.REFCLK0_P: track 0.71 -> 8.97 mm
- net /FPGA MGT Interface/GTX118.RX3_N: track 0.71 -> 8.66 mm
- net /FPGA MGT Interface/GTX118.REFCLK1_N: track 0.71 -> 8.66 mm
- net /FPGA MGT Interface/GTX118.REFCLK0_N: track 0.71 -> 8.66 mm
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Other:
- copper layers 2 -> 10
