File: fpga-bank-14-15.kicad_sch (KiCad schematic)
At the start: 23 parts, among them U1 XC7K410T-2FFG900I

Commit message: Fix project name, update README, cleanup files
Parts:
- NT10, NT11, NT12, NT13, NT14, NT20, NT9: symbol K410T-devboard:Net-Tie_2 -> k410t-devboard:Net-Tie_2
Changed lines of the file:
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@@
 	)
 	(symbol
-		(lib_id "K410T-devboard:Net-Tie_2")
+		(lib_id "k410t-devboard:Net-Tie_2")
 		(at 149.86 115.57 0)
 		(mirror y)
@@
 		)
 		(instances
-			(project "K410T-devboard"
+			(project "k410t-devboard"
 				(path "/c1489e7c-896d-4046-acd4-3929998e87dc/429ead79-12f0-47b8-8167-aee96d75a5d4"
 					(reference "NT11")
@@
 	)
 	(symbol
-		(lib_id "K410T-devboard:Net-Tie_2")
+		(lib_id "k410t-devboard:Net-Tie_2")
 		(at 149.86 102.87 0)
 		(mirror y)
@@
 		)
 		(instances
-			(project "K410T-devboard"
+			(project "k410t-devboard"
 				(path "/c1489e7c-896d-4046-acd4-3929998e87dc/429ead79-12f0-47b8-8167-aee96d75a5d4"
 					(reference "NT9")
@@
 		)
 		(instances
-			(project "K410T-devboard"
+			(project "k410t-devboard"
 				(path "/c1489e7c-896d-4046-acd4-3929998e87dc/429ead79-12f0-47b8-8167-aee96d75a5d4"
 					(reference "C37")
@@
 		)
 		(instances
-			(project "K410T-devboard"
+			(project "k410t-devboard"
 				(path "/c1489e7c-896d-4046-acd4-3929998e87dc/429ead79-12f0-47b8-8167-aee96d75a5d4"
 					(reference "#PWR011")
@@
 		)
 		(instances
-			(project "K410T-devboard"
+			(project "k410t-devboard"
 				(path "/c1489e7c-896d-4046-acd4-3929998e87dc/429ead79-12f0-47b8-8167-aee96d75a5d4"
 					(reference "#PWR012")
@@
 		)
 		(instances
-			(project "K410T-devboard"
+			(project "k410t-devboard"
 				(path "/c1489e7c-896d-4046-acd4-3929998e87dc/429ead79-12f0-47b8-8167-aee96d75a5d4"
 					(reference "R338")
@@
 		)
 		(instances
-			(project "K410T-devboard"
+			(project "k410t-devboard"
 				(path "/c1489e7c-896d-4046-acd4-3929998e87dc/429ead79-12f0-47b8-8167-aee96d75a5d4"
 					(reference "C42")
@@
 		)
 		(instances
-			(project "K410T-devboard"
+			(project "k410t-devboard"
 				(path "/c1489e7c-896d-4046-acd4-3929998e87dc/429ead79-12f0-47b8-8167-aee96d75a5d4"
 					(reference "C31")
@@
 		)
 		(instances
-			(project "K410T-devboard"
+			(project "k410t-devboard"
 				(path "/c1489e7c-896d-4046-acd4-3929998e87dc/429ead79-12f0-47b8-8167-aee96d75a5d4"
 					(reference "C19")
@@
 		)
 		(instances
-			(project "K410T-devboard"
+			(project "k410t-devboard"
 				(path "/c1489e7c-896d-4046-acd4-3929998e87dc/429ead79-12f0-47b8-8167-aee96d75a5d4"
 					(reference "U1")
@@
 		)
 		(instances
-			(project "K410T-devboard"
+			(project "k410t-devboard"
 				(path "/c1489e7c-896d-4046-acd4-3929998e87dc/429ead79-12f0-47b8-8167-aee96d75a5d4"
 					(reference "C38")
@@
 		)
 		(instances
-			(project "K410T-devboard"
+			(project "k410t-devboard"
 				(path "/c1489e7c-896d-4046-acd4-3929998e87dc/429ead79-12f0-47b8-8167-aee96d75a5d4"
 					(reference "C26")
@@
 	)
 	(symbol
-		(lib_id "K410T-devboard:Net-Tie_2")
+		(lib_id "k410t-devboard:Net-Tie_2")
 		(at 149.86 113.03 0)
 		(mirror y)
@@
 		)
 		(instances
-			(project "K410T-devboard"
+			(project "k410t-devboard"
 				(path "/c1489e7c-896d-4046-acd4-3929998e87dc/429ead79-12f0-47b8-8167-aee96d75a5d4"
 					(reference "NT10")
@@
 	)
 	(symbol
-		(lib_id "K410T-devboard:Net-Tie_2")
+		(lib_id "k410t-devboard:Net-Tie_2")
 		(at 127 120.65 0)
 		(mirror y)
@@
 		)
 		(instances
-			(project "K410T-devboard"
+			(project "k410t-devboard"
 				(path "/c1489e7c-896d-4046-acd4-3929998e87dc/429ead79-12f0-47b8-8167-aee96d75a5d4"
 					(reference "NT20")
@@
 		)
 		(instances
-			(project "K410T-devboard"
+			(project "k410t-devboard"
 				(path "/c1489e7c-896d-4046-acd4-3929998e87dc/429ead79-12f0-47b8-8167-aee96d75a5d4"
 					(reference "C20")
@@
 	)
 	(symbol
-		(lib_id "K410T-devboard:Net-Tie_2")
+		(lib_id "k410t-devboard:Net-Tie_2")
 		(at 127 97.79 0)
 		(mirror y)
@@
 		)
 		(instances
-			(project "K410T-devboard"
+			(project "k410t-devboard"
 				(path "/c1489e7c-896d-4046-acd4-3929998e87dc/429ead79-12f0-47b8-8167-aee96d75a5d4"
 					(reference "NT14")
@@
 		)
 		(instances
-			(project "K410T-devboard"
+			(project "k410t-devboard"
 				(path "/c1489e7c-896d-4046-acd4-3929998e87dc/429ead79-12f0-47b8-8167-aee96d75a5d4"
 					(reference "C13")
@@
 		)
 		(instances
-			(project "K410T-devboard"
+			(project "k410t-devboard"
 				(path "/c1489e7c-896d-4046-acd4-3929998e87dc/429ead79-12f0-47b8-8167-aee96d75a5d4"
 					(reference "C32")
@@
 		)
 		(instances
-			(project "K410T-devboard"
+			(project "k410t-devboard"
 				(path "/c1489e7c-896d-4046-acd4-3929998e87dc/429ead79-12f0-47b8-8167-aee96d75a5d4"
 					(reference "C6")
@@
 		)
 		(instances
-			(project "K410T-devboard"
+			(project "k410t-devboard"
 				(path "/c1489e7c-896d-4046-acd4-3929998e87dc/429ead79-12f0-47b8-8167-aee96d75a5d4"
 					(reference "C14")
@@
 		)
 		(instances
-			(project "K410T-devboard"
+			(project "k410t-devboard"
 				(path "/c1489e7c-896d-4046-acd4-3929998e87dc/429ead79-12f0-47b8-8167-aee96d75a5d4"
 					(reference "#PWR0477")
@@
 		)
 		(instances
-			(project "K410T-devboard"
+			(project "k410t-devboard"
 				(path "/c1489e7c-896d-4046-acd4-3929998e87dc/429ead79-12f0-47b8-8167-aee96d75a5d4"
 					(reference "C43")
@@
 	)
 	(symbol
-		(lib_id "K410T-devboard:Net-Tie_2")
+		(lib_id "k410t-devboard:Net-Tie_2")
 		(at 149.86 118.11 0)
 		(mirror y)
@@
 		)
 		(instances
-			(project "K410T-devboard"
+			(project "k410t-devboard"
 				(path "/c1489e7c-896d-4046-acd4-3929998e87dc/429ead79-12f0-47b8-8167-aee96d75a5d4"
 					(reference "NT12")
@@
 		)
 		(instances
-			(project "K410T-devboard"
+			(project "k410t-devboard"
 				(path "/c1489e7c-896d-4046-acd4-3929998e87dc/429ead79-12f0-47b8-8167-aee96d75a5d4"
 					(reference "C5")
@@
 		)
 		(instances
-			(project "K410T-devboard"
+			(project "k410t-devboard"
 				(path "/c1489e7c-896d-4046-acd4-3929998e87dc/429ead79-12f0-47b8-8167-aee96d75a5d4"
 					(reference "C25")
@@
 		)
 		(instances
-			(project "K410T-devboard"
+			(project "k410t-devboard"
 				(path "/c1489e7c-896d-4046-acd4-3929998e87dc/429ead79-12f0-47b8-8167-aee96d75a5d4"
 					(reference "#PWR014")
@@
 	)
 	(symbol
-		(lib_id "K410T-devboard:Net-Tie_2")
+		(lib_id "k410t-devboard:Net-Tie_2")
 		(at 127 95.25 0)
 		(mirror y)
@@
 		)
 		(instances
-			(project "K410T-devboard"
+			(project "k410t-devboard"
 				(path "/c1489e7c-896d-4046-acd4-3929998e87dc/429ead79-12f0-47b8-8167-aee96d75a5d4"
 					(reference "NT13")
@@
 		)
 		(instances
-			(project "K410T-devboard"
+			(project "k410t-devboard"
 				(path "/c1489e7c-896d-4046-acd4-3929998e87dc/429ead79-12f0-47b8-8167-aee96d75a5d4"
 					(reference "#PWR016")
